File: connectors.kicad_sch (KiCad schematic)
At the start: 0 parts

Commit message: Added Connectors; added hierarchical labels connections
Parts:
- added J1: USB_A, symbol Connector:USB_A
- added J2: IN_R connector, symbol Connector_Generic:Conn_01x03
- added J3: MIC connector, symbol Connector_Generic:Conn_01x02
Connections:
- new net D+: J1.3 (D+)
- new net D-: J1.2 (D-)
- new net GND: J1.4 (GND), J2.2 (Pin_2), J3.2 (Pin_2)
- new net IN_R: J2.3 (Pin_3)
- new net MIC+: J3.1 (Pin_1)
- new net VBUS: J1.1 (VBUS)
- new net VCC: J2.1 (Pin_1)
- no-connect marks 0 -> 1
Other:
- company: (none) -> Maksym Rybalskyi <MaxDespairon@gmail.com>
- title: (none) -> Connectors

Commit message: Add missing PCM2906 components; Partially Implement PCB
Parts:
- J1: footprint (none) -> Connector_USB:USB3_A_Molex_48393-001
- J2: footprint (none) -> Connector_PinHeader_1.27mm:PinHeader_1x03_P1.27mm_Vertical
- J3: footprint (none) -> Connector_PinHeader_1.27mm:PinHeader_1x02_P1.27mm_Vertical
Changed lines of the file:
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@@
 		(dnp no)
 		(fields_autoplaced yes)
-		(property "Reference" "#PWR023"
+		(property "Reference" "#PWR022"
 			(at 102.87 85.09 0)
 			(effects
@@
 			(project "kicad_mic_amp"
 				(path "/eb1afd54-626c-4526-850f-b0511eb9dc59/9643d481-3898-40ec-96ff-319a188d3022"
-					(reference "#PWR023")
+					(reference "#PWR022")
 					(unit 1)
 				)
@@
 			)
 		)
-		(property "Footprint" ""
+		(property "Footprint" "Connector_PinHeader_1.27mm:PinHeader_1x02_P1.27mm_Vertical"
 			(at 102.87 123.19 0)
 			(effects
@@
 			)
 		)
-		(property "Footprint" ""
+		(property "Footprint" "Connector_USB:USB3_A_Molex_48393-001"
 			(at 106.68 69.85 0)
 			(effects
@@
 		(dnp no)
 		(fields_autoplaced yes)
-		(property "Reference" "#PWR020"
+		(property "Reference" "#PWR019"
 			(at 87.63 104.14 0)
 			(effects
@@
 			(project ""
 				(path "/eb1afd54-626c-4526-850f-b0511eb9dc59/9643d481-3898-40ec-96ff-319a188d3022"
-					(reference "#PWR020")
+					(reference "#PWR019")
 					(unit 1)
 				)
@@
 			)
 		)
-		(property "Footprint" ""
+		(property "Footprint" "Connector_PinHeader_1.27mm:PinHeader_1x03_P1.27mm_Vertical"
 			(at 102.87 97.79 0)
 			(effects
@@
 		(dnp no)
 		(fields_autoplaced yes)
-		(property "Reference" "#PWR022"
+		(property "Reference" "#PWR023"
 			(at 114.3 67.31 0)
 			(effects
@@
 			(project ""
 				(path "/eb1afd54-626c-4526-850f-b0511eb9dc59/9643d481-3898-40ec-96ff-319a188d3022"
-					(reference "#PWR022")
+					(reference "#PWR023")
 					(unit 1)
 				)
@@
 		(dnp no)
 		(fields_autoplaced yes)
-		(property "Reference" "#PWR019"
+		(property "Reference" "#PWR020"
 			(at 95.25 99.06 0)
 			(effects
@@
 			(project ""
 				(path "/eb1afd54-626c-4526-850f-b0511eb9dc59/9643d481-3898-40ec-96ff-319a188d3022"
-					(reference "#PWR019")
-					(unit 1)
-				)
+					(reference "#PWR020")
+					(unit 1)
+				)
